File: Board Files/Motherboard.kicad_sch (KiCad schematic)
At the start: 121 parts, among them P1 72-Pin Connector, P2 EXP-Connector, P3 MOD RF, P4 Controller Input, P5 Controller Input, P6 PWR/RST IN, Q1 2SA937, Q2 2SC2021, Q3 2SC2021, U1 6116 (WRAM), U10 CIC, U2 74HC373, U3 74HC139, U4 6116 (VRAM), U5 RP2C02 PPU, U6 RP2A03 CPU, U7 40H368 (CI), U8 40H368 (CII), U9 74LS04, X1 21.477272 MHz, X2 4MHz

Commit message: feat: updated trimmer cap footprint
Parts:
- TC1: footprint NESRE:TrimmerCap-THT -> NESRE:Trimmer_Cap_THT_5_5
Changed lines of the file:
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@@
 			)
 		)
-		(property "Footprint" "NESRE:TrimmerCap-THT"
+		(property "Footprint" "NESRE:Trimmer_Cap_THT_5_5"
 			(at 66.04 191.77 0)
 			(effects
